File: Tractive System Light Control Board.brd (EAGLE design)
At the start: 160 x 100 mm, 131 parts, among them J2 MOLEX_CLICKMATE-2-VERTICAL, J3 MOLEX_CLICKMATE-2-VERTICAL, Q1 BSS138, Q100 FQD2N100, Q101 MMBT2222A, Q102 STP5N60M2, Q12 FQD3P50, Q5 BSS138, T1 WURTH-7491181112, U1 ISO7221, U10 TPS562219, U100 LM5022, U14 LM139, U2 TPS562219, U3 CD4069UB-SOIC, U36 LTC1155, U37 CSD17506Q5A, U4 CD4071B, U44 TL7712A-SOIC, U6 LTC1155, U8 CSD17506Q5A

Commit message: Added 55 Timer schematics and DC DC Converter
Parts:
- removed C33, C34: 0.1uF, adafruit:C0805
- removed C35, C36: 1uF, rcl:C0805
- removed Q5: BSS138, FormE:BSS138
- removed R53, R54: 10k, rcl:R0805
- removed R55: 100, rcl:R0805
- removed R56: 2.2K, rcl:R0805
- removed S2: TE-FSM4JSMATR, FormE:TE-FSM4JSMATR
- removed TP38, TP39, TP40: PTR1TP20R, testpad:TP20R
- removed U3: CD4069UB-SOIC, FormE:D14
- removed U4: CD4071B, FormE:PW14
- removed U44: TL7712A-SOIC, FormE:D8
- added H3: (no value), FormE:MOLEX_MX120G
- added J4: MOLEX_CLICKMATE-2-VERTICAL, FormE:MOLEX-CLIKMATE-2-VERTICAL-HEADER
- added U9: SN74LVC1G86, FormE:LITTLE_LOGIC_BASIC
- J1: value (none) -> MOLEX_CLICKMATE-2-VERTICAL; device FormE:MOLEX-PICOLOCK-4PIN-504050-0491 -> FormE:MOLEX-CLIKMATE-2-VERTICAL-HEADER
- T2: device FormE:ICM7555,56 -> FormE:LMC555
- moved J3 86.4 mm to (-112.4, -5.71)
- moved J1 73.1 mm to (-136.5, -5.71)
- moved C20 3.18 mm to (86.4, 15.2)
- moved C1 3.17 mm to (86.4, 10.2)
- moved LED2 3.17 mm to (84.5, 7.62)
- moved R27 3.17 mm to (88.3, 7.62)
- moved C19 3.17 mm to (86.4, 12.7)
- moved L2 3.17 mm to (78.1, 12.1)
Connections:
- net N$80 renamed 60V_CHECK
- removed net +3V3: Q5.G, R54.2, R56.1
- removed net AMS_DIGITAL_OV-12V: J1.1, U3.1
- removed net LED_CONTROL: TP20.TP, U37.1, U37.2, U37.3
- removed net MCU_RESET: C36.1, R55.1, R56.2, TP39.TP, U44.2
- removed net N$26: C33.2, U44.3
- removed net N$27: C34.2, U44.1
- removed net N$63: Q5.S, R54.1, U35.5
- removed net N$65: Q5.D, R53.1, TP38.TP, U44.5
- removed net N$66: R55.2, S2.1, S2.2
- removed net POR: TP40.TP, U35.6
- removed net VDD: C35.1, R53.2, U44.7, U44.8
- new net AMS_CONTACTOR: J4.2
- new net LED_CONTROL_12V: H3.10, H3.11, H3.12, H3.7, H3.8, H3.9, TP20.TP, U37.1, U37.2, U37.3
- net +5V: no longer U3.14
- net +5V/1: now also U9.5; no longer U4.14
- net AMS_DIGITAL_+12V_INVERTED_HV: now also U9.2; no longer U4.2
- net AMS_DIGITAL_+12V_INVERTED_LV: no longer U3.2
- net GND: now also J3.2; no longer J1.3, U3.7
- net GND1: now also H3.1, H3.2, H3.3, H3.4, H3.5, H3.6, J2.1, U9.3; no longer C33.1, C34.1, C35.2, C36.2, S2.3, S2.4, U4.7, U44.4
- net HV_INDICATOR_OUTPUT_+12V: now also U9.1; no longer U4.1
- net N$9: now also U9.4; no longer U4.3
- net V+: now also J1.1, J1.2; no longer J2.1
- net VCC: now also J3.1; no longer J1.2
Routing:
- net LED_CONTROL_12V: track 0.00 -> 1.96 mm, vias 0 -> 4
- net LED_CONTROL: track 1.96 -> 0.00 mm, vias 4 -> 0
- net 555_TIMER_SUPPLY: track 24.7 -> 26.5 mm
- net N$6: track 31.0 -> 32.5 mm
- net N$19: track 15.7 -> 16.9 mm
- net N$15: track 9.13 -> 10.3 mm
- net +5V/1: track 15.5 -> 14.6 mm
- net N$20: track 18.2 -> 18.9 mm
- net N$5: track 11.6 -> 12.3 mm
- net GND: vias 32 -> 26
- added copper zone on layer 1, net LED_CONTROL_12V
- removed copper zone on layer 1, net LED_CONTROL

Commit message: Mid-design change, about to start deleting things
Parts:
- removed LED10, LED11, LED3, LED9: (no value), FormE:SMARTLED-TTW
- added LED4, LED6, LED7: (no value), FormE:SMARTLED-TTW
- added LED5: GREEN, FormE:CHIPLED_0805
- added R18, R19, R21, R22, R23: 10k, adafruit:R0805
- added U3: SN74LVC1G04DRL, FormE:LITTLE_LOGIC_BASIC_DRL
- added U38: LM124, FormE:D14
- R2: value 54.9k -> 33.2K
- R9: value 100 -> 1K
- U9: value SN74LVC1G86 -> SN74LVC1G86DRL; device FormE:LITTLE_LOGIC_BASIC -> FormE:LITTLE_LOGIC_BASIC_DRL
- moved R4 266.2 mm to (-141.0, -74.3), turned to 0 degrees
- moved C2 264.9 mm to (-141.0, -62.9), turned to 0 degrees
- moved C7 261.5 mm to (-141.0, -68.6)
- moved R5 258.9 mm to (-135.3, -74.3), turned to 0 degrees
- moved LED8 257.3 mm to (-161.3, -92.7), turned to 0 degrees
- moved C8 256.2 mm to (-134.6, -68.6)
- moved C3 254.2 mm to (-127.0, -62.9), turned to 0 degrees
- moved C9 251.0 mm to (-128.3, -68.6)
- moved C4 250.6 mm to (-120.7, -62.9), turned to 0 degrees
- moved C5 250.1 mm to (-134.6, -55.9), turned to 0 degrees
- moved C6 248.8 mm to (-134.0, -62.9), turned to 0 degrees
- moved L1 244.9 mm to (-137.8, -45.7), turned to 0 degrees
- moved U2 242.9 mm to (-128.9, -44.5), turned to 0 degrees
- moved R2 238.7 mm to (-125.7, -55.9), turned to 0 degrees
- moved R3 238.2 mm to (-121.9, -68.6), turned to 0 degrees
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Connections:
- net SW_5V1 renamed SW_5V2
- removed net N$46: LED8.A@1, LED9.C@1
- removed net N$47: R20.2, R24.2, U14.14
- removed net N$50: LED10.A@1, LED11.C@1
- removed net N$51: LED10.C@1, LED9.A@1
- removed net N$52: LED11.A@1, R9.2
- new net +3V3: C7.1, C8.1, C9.1, L1.P$2, LED5.A, R2.2
- new net HV_INDICATOR_SIGNAL: R20.2, R24.2, U3.4
- new net N$18: R18.2, R19.1
- new net N$21: LED4.C@1, R9.2
- new net N$22: LED4.A@1, LED6.C@1
- new net N$24: LED6.A@1, LED7.C@1
- new net N$25: LED7.A@1, LED8.C@1
- new net N$26: R19.2, R21.1
- new net N$27: R21.2, R22.1
- new net N$30: R22.2, R23.1
- new net N$35: U3.2, U38.8
- net +5V: no longer C7.1, C8.1, C9.1, L1.P$2, LED3.A@1, R2.2
- net +5V/1: now also LED8.A@1, U3.5
- net FILTERED_BATT_VOLTAGE_FB: now also U38.10; no longer U14.8
- net GND1: now also R23.2, U3.3
- net HV_INDICATOR_OUTPUT_+12V: no longer R9.1
- net N$2: now also LED5.C; no longer LED3.C@1
- net N$48: now also U38.9; no longer U14.9
- net N$60: now also R9.1; no longer LED8.C@1
- net V+: now also R18.1
Routing:
- net N$47: track 18.5 -> 0.00 mm, vias 2 -> 0
- net HV_INDICATOR_SIGNAL: track 0.00 -> 17.8 mm, vias 0 -> 2
- net FILTERED_BATT_VOLTAGE_FB: track 11.7 -> 2.54 mm
- net N$1: track 8.37 -> 0.00 mm, vias 2 -> 0
- net HV_INDICATOR_OUTPUT_+12V: track 7.40 -> 0.00 mm
- net VFB_5V1: track 7.25 -> 0.00 mm
- net VBST_5V1: track 5.57 -> 0.00 mm
- net GND: track 5.03 -> 0.00 mm, vias 26 -> 24
- net SS_5V1: track 2.66 -> 0.00 mm
- net VCC: track 11.6 -> 9.17 mm, vias 12 -> 11
- net N$2: track 2.31 -> 0.00 mm
- net SW_5V2: track 2.31 -> 0.00 mm, vias 11 -> 0
- net N$48: track 22.1 -> 20.2 mm
- net N$51: track 1.91 -> 0.00 mm
- net N$46: track 1.91 -> 0.00 mm
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- added copper zone on layer 1, net SW_5V1
- added copper zone on layer 16, net SW_5V1
- removed copper zone on layer 1, net SW_5V2
- removed copper zone on layer 16, net SW_5V2

Commit message: Schematic Done
Parts:
- removed C1, C19, C20: 22uF, adafruit:C0805
- removed C10: DNP, adafruit:C0805K
- removed C100, C101: 0.047uF, adafruit:C1812K
- removed C102: 0.022uF, adafruit:C0805K
- removed C103: 4.7uF, adafruit:C1210K
- removed C104: 1uF, adafruit:C0805K
- removed C105: 680pF, adafruit:C0805K
- removed C106: 330pF, adafruit:C0805K
- removed C107: 6800pF, adafruit:C0805K
- removed C111: 100uF, adafruit:PANASONIC_F
- removed C12, C16: 0.1uF, adafruit:C0805
- removed C121: 0.33uF, adafruit:C0805K
- removed C13, C14: 10uF, adafruit:C0805
- removed C15: 8200pF, adafruit:C0805
- removed C17: 3.3uF, adafruit:C1210K
- removed D100, D5: CMZ5931B, FormE:CMZ59
- removed D101: ES1D, FormE:ES1D
- removed D105, D3: BAV21W, FormE:BAV21W
- removed D110: CMZ5918B, FormE:CMZ59
- removed F1: 0805L020, FormE:PTC-FUSE-0805
- removed F2: 0485.500DR, FormE:LITTELFUSE_485
- removed H3: (no value), FormE:MOLEX_MX120G
- removed J3, J4: MOLEX_CLICKMATE-2-VERTICAL, FormE:MOLEX-CLIKMATE-2-VERTICAL-HEADER
- removed L2: 4.7uH, FormE:SRP6540
- removed Q100: FQD2N100, FormE:FQD2N100
- removed Q101: MMBT2222A, FormE:SOT-23
- removed Q102: STP5N60M2, FormE:STP3N150
- removed Q12: FQD3P50, FormE:FQD3P50
- removed R100, R101, R102, R103, R104, R105, R47: 1M, adafruit:R0805
- removed R106, R113: 20.5k, adafruit:R0805
- removed R107: 8.25k, adafruit:R0805
- removed R108: 499, adafruit:R0805
- removed R109: 1.05k, adafruit:R0805
- removed R110: 17.4k, adafruit:R0805
- removed R111: 2k, adafruit:R0805
- removed R112: 24.9, adafruit:R0805
- removed R114: 243k, adafruit:R0805
- removed R115: 0.82, adafruit:R1210
- removed R116: 2M, adafruit:R0805
- removed R117: 10k, adafruit:R1210
- removed R121: 205k, adafruit:R0805
- removed R25, R26: 10K, adafruit:R0805
- removed R27: 1K, adafruit:R0805
- removed R7: 4.7k, adafruit:R0805
- removed R8: 0, adafruit:R0805
- removed TP20: PTR1TP20R, testpad:TP20R
- removed U$1: AAVID-579302B00000G, FormE:AAVID-579302B00000G
- removed U10: TPS562219, FormE:TPS562219
- removed U100: LM5022, FormE:LM5022
- added C72, C73: 10uF, adafruit:C0805
- added C90, C91: 10uF, rcl:C1206
- added D33, D34: MBR0520LT3G, FormE:SOD-123
- added D35: MM3Z5V1B, FormE:SOD323F
- added H1: (no value), FormE:MOLEX-CLIKMATE-8-VERTICAL-HEADER
- added R72: 47R, rcl:R0805
- added TP2: PTR1TP20R, testpad:TP20R
- added U12: SN6501DBVR, FormE:SN6501DBV
- added U21: LM1085IS, FormE:TO-263
- LED2: value (none) -> GREEN; device FormE:SMARTLED-TTW -> FormE:CHIPLED_0805
- R1: value 54.9k -> 1K
- R2: value 33.2K -> 54.9K
- R6: value 470k -> 0.007
- T1: value WURTH-7491181112 -> 750313734; device FormE:WURTH-7491181112 -> FormE:WURTH-750313734
- moved T1 333.0 mm to (-155.6, -148.6), turned to 0 degrees
- moved R1 320.2 mm to (-154.9, -194.9), turned to 0 degrees
- moved LED2 314.8 mm to (-160.7, -189.9), turned to 0 degrees
- moved R6 289.6 mm to (-155.6, -187.3), turned to 0 degrees
Connections:
- removed net +3V3: C7.1, C8.1, C9.1, L1.P$2, LED5.A, R2.2
- removed net 60V_CHECK: C100.1, C101.1, D5.1, Q12.S, R100.2, R103.2, R106.2, R6.2, T1.P$1
- removed net AMS_CONTACTOR: J4.2
- removed net AMS_DIGITAL_+12V_INVERTED_HV: U9.2
- removed net AMS_DIGITAL_+12V_INVERTED_LV: U1.P$3
- removed net BATT_VOLTAGE_FB: R6.1, R7.2, R8.1
- removed net COMP: C106.1, R107.1, U100.P$3, U100.P3
- removed net CS: R109.1, R116.2, U100.P$8, U100.P8
- removed net FB: C106.2, C107.2, R110.1, R111.2, U100.P$2, U100.P2
- removed net FILTERED_BATT_VOLTAGE_FB: C10.1, R8.2, U38.10
- removed net HV_INDICATOR_OUTPUT_+12V: U9.1
- removed net HV_INDICATOR_SIGNAL: R20.2, R24.2, U3.4
- removed net N$10: R103.1, R104.2, R116.1
- removed net N$11: R104.1, R105.2
- removed net N$12: R101.1, R102.2
- removed net N$14: C121.1, D110.1, Q101.B, R102.1, R121.2
- removed net N$23: R26.2, U10.7
- removed net N$28: LED2.C@1, R27.2
- removed net N$29: D105.ANODE, R112.1
- removed net N$30: R22.2, R23.1
- removed net N$32: Q102.S, R108.2, R115.2
- removed net N$33: Q102.D, T1.P$5
- removed net N$34: C105.1, R108.1, R109.2
- removed net N$37: Q100.D, R106.1
- removed net N$38: D101.2, T1.P$6
- removed net N$4: D105.CATHODE, D3.ANODE, R110.2
- removed net N$7: R100.1, R101.2
- removed net N$81: D5.2, Q12.G, R47.2
- removed net N$82: D101.1, F1.P$1
- removed net N$83: F2.P$2, Q12.D
- removed net OUT: Q102.G, U100.P$5, U100.P5
- removed net RT: R114.2, U100.P$9, U100.P9
- removed net SS: C102.1, U100.P$10, U100.P10
- removed net SS_5V: C15.1, U10.5
- removed net SW_5V: C16.2, L2.P$1, U10.2
- removed net UVLO: Q101.E, R113.2, U100.P$7, U100.P7
- removed net VBST_5V: C16.1, U10.8
- removed net VFB_5V: R1.1, R25.2, U10.6
- removed net VIN: C103.1, D3.CATHODE, Q100.S, Q101.C, U100.P$1, U100.P1
- new net 12V_CURRENT_SENSE+: C73.1, R6.1, U21.2, U21.GND, U21.GND1
- new net AMS_CONTACTOR_INVERTED: H1.8, U9.2
- new net BATT_V_REFERENCE: R22.2, R23.1, U38.10
- new net HV_INDICATOR_SIGNAL_HV: R20.2, R24.2, U1.P$2, U3.4
- new net HV_INDICATOR_SIGNAL_LV: U1.P$7, U9.1
- new net N$40: T1.3, U12.1
- new net N$41: D33.A, T1.6
- new net N$43: C90.1, D33.K, D34.K, R72.1
- new net N$45: D34.A, T1.4
- net +12V: now also LED2.A, R6.2; no longer C111.+, C17.1, F1.P$2, R112.2, R117.2
- net +5V: now also C7.1, C8.1, C9.1, L1.P$2, LED5.A, R2.2, T1.2, U1.P$8, U12.2; no longer U1.P$1
- net +5V/1: now also C91.1, D35.CATHODE, R72.2, U1.P$1; no longer C1.1, C19.1, C20.1, L2.P$2, LED2.A@1, R1.2, U1.P$8
- net GND: now also C72.2, C73.2, H1.2, H1.5, H1.6, R1.1, U1.P$5, U12.4, U12.5, U21.1; no longer C1.2, C12.2, C13.2, C14.2, C19.2, C20.2, J3.2, R27.1, U1.P$4
- net GND1: now also C90.2, C91.2, D35.ANODE, T1.5, U1.P$4; no longer C10.2, C100.2, C101.2, C102.2, C103.2, C104.2, C105.2, C111.-, C121.2, C15.2, C17.2, D100.2, D110.2, H3.1, H3.2, H3.3, H3.4, H3.5, H3.6, R111.1, R113.1, R114.1, R115.1, R117.1, R121.1, R25.1, R47.1, R7.1, T1.P$9, U1.P$5, U10.1, U100.P$6, U100.P6
- net LED_CONTROL_12V: now also H1.3, H1.4, TP2.TP; no longer H3.10, H3.11, H3.12, H3.7, H3.8, H3.9, TP20.TP
- net N$13: now also LED2.C, R1.2; no longer D100.1, Q100.G, R105.1
- net N$31: now also T1.1, U12.3; no longer C107.1, R107.2
- net V+: no longer F2.P$1
- net VCC: now also C72.1, H1.7, U21.3; no longer C104.1, C12.1, C13.1, C14.1, J3.1, R26.1, U10.3, U100.P$4, U100.P4
Routing:
- net N$10: track 38.2 -> 0.00 mm, vias 2 -> 0
- net GND1: track 50.7 -> 28.2 mm, vias 68 -> 60
- net HV_INDICATOR_SIGNAL_HV: track 0.00 -> 17.8 mm, vias 0 -> 2
- net HV_INDICATOR_SIGNAL: track 17.8 -> 0.00 mm, vias 2 -> 0
- net UVLO: track 16.0 -> 0.00 mm, vias 2 -> 0
- net CS: track 10.3 -> 0.00 mm
- net VCC: track 9.17 -> 0.00 mm, vias 11 -> 10
- net N$23: track 8.37 -> 0.00 mm, vias 2 -> 0
- net COMP: track 8.08 -> 0.00 mm
- net VFB_5V: track 6.85 -> 0.00 mm
- net SS: track 5.79 -> 0.00 mm
- net VBST_5V: track 5.57 -> 0.00 mm
- net N$34: track 5.46 -> 0.00 mm
- net VIN: track 5.28 -> 0.00 mm, vias 7 -> 6
- net BATT_VOLTAGE_FB: track 5.08 -> 0.00 mm
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
Commit message: Layout Done: Need graphic for HV, maybe logo in bottom right corner?
Parts:
- removed U14: LM139, FormE:D14
- removed U35: (no value), FormE:SOIC-14
- moved H1 330.5 mm to (83.8, 22.2), turned to 90 degrees
- moved TP2 306.2 mm to (76.8, 22.2)
- moved C73 305.4 mm to (58.4, 17.1)
- moved LED2 298.5 mm to (60.3, 10.8), turned to 90 degrees
- moved R1 296.0 mm to (60.3, 8.26), turned to 180 degrees
- moved R6 295.6 mm to (60.3, 14.6)
- moved U12 282.5 mm to (48.3, 33.7), turned to 270 degrees
- moved U21 276.9 mm to (48.9, 8.89), turned to 180 degrees
- moved C72 268.5 mm to (40.6, 3.17), turned to 270 degrees
- moved T1 265.0 mm to (36.8, 33.7), turned to 180 degrees
- moved R72 262.3 mm to (19.1, 27.3), turned to 270 degrees
- moved D34 261.8 mm to (24.8, 26.0), turned to 90 degrees
- moved C90 251.4 mm to (21.6, 21.0), turned to 270 degrees
- moved D35 247.3 mm to (15.9, 21.0), turned to 270 degrees
- moved C91 245.2 mm to (19.1, 21.0), turned to 270 degrees
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Connections:
- net +12V: no longer U35.14
- net +5V: now also R50.2, U6.1, U6.6, U8.5, U8.6, U8.7, U8.8, U8.PAD, U8.PAD1, U8.VIA1, U8.VIA2, U8.VIA3, U8.VIA4, U8.VIA5, U8.VIA6, U8.VIA7, U8.VIA8, U8.VIA9, U9.5
- net +5V/1: now also U38.4; no longer R50.2, U14.3, U6.1, U6.6, U8.5, U8.6, U8.7, U8.8, U8.PAD, U8.PAD1, U8.VIA1, U8.VIA2, U8.VIA3, U8.VIA4, U8.VIA5, U8.VIA6, U8.VIA7, U8.VIA8, U8.VIA9, U9.5
- net AMS_CONTACTOR_INVERTED: now also H1.4; no longer H1.8
- net GND: now also C11.-, C18.1, H1.8, R12.1, R17.1, T2.P$5, U36.3, U6.3, U9.3; no longer H1.6
- net GND1: now also U38.11; no longer C11.-, C18.1, R12.1, R17.1, T2.P$5, U14.12, U35.7, U36.3, U6.3, U9.3
- net LED_CONTROL_12V: now also H1.6, H1.7; no longer H1.3, H1.4
- net VCC: now also H1.1; no longer H1.7
Routing:
- net AMS_CONTACTOR_INVERTED: track 0.00 -> 47.4 mm, vias 0 -> 2
- net GND: track 0.00 -> 28.7 mm, vias 24 -> 41
- net 555_TIMER_OUTPUT: track 18.3 -> 40.2 mm, vias 0 -> 3
- net BATT_V_REFERENCE: track 0.00 -> 20.8 mm
- net HV_INDICATOR_SIGNAL_HV: track 17.8 -> 37.1 mm
- net N$45: track 0.00 -> 17.7 mm
- net N$49: track 19.8 -> 3.27 mm, vias 2 -> 0
- net N$48: track 20.2 -> 5.90 mm, vias 2 -> 0
- net N$43: track 0.00 -> 10.5 mm
- net GND1: track 28.2 -> 37.3 mm, vias 60 -> 13
- net N$35: track 0.00 -> 8.95 mm, vias 0 -> 2
- net N$1: track 0.00 -> 7.73 mm, vias 0 -> 2
- net +5V: track 0.00 -> 7.59 mm, vias 6 -> 24
- net VFB_5V1: track 0.00 -> 6.85 mm
- net N$41: track 0.00 -> 5.93 mm
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- added copper zone on layer 15, net +12V
- added copper zone on layer 15, net +5V
- added copper zone on layer 1, net 12V_CURRENT_SENSE+
- added copper zone on layer 1, net 555_TIMER_SUPPLY
- added copper zone on layer 2, net GND
- added copper zone on layer 1, net SW_5V2
- added copper zone on layer 16, net SW_5V2
- added copper zone on layer 1, net V+
- added copper zone on layer 15, net VCC
- removed copper zone on layer 1, net 60V_CHECK
- removed copper zone on layer 16, net 60V_CHECK
- removed copper zone on layer 1, net FB
- removed copper zone on layer 16, net GND1
- removed copper zone on layer 1, net N$10
- removed copper zone on layer 1, net N$11
- removed copper zone on layer 1, net N$12
- removed copper zone on layer 16, net N$17
- removed copper zone on layer 1, net N$29
- removed copper zone on layer 1, net N$32
- removed copper zone on layer 1, net N$33
- removed copper zone on layer 1, net N$38
- removed copper zone on layer 1, net N$4
- removed copper zone on layer 1, net N$7
- removed copper zone on layer 1, net N$82
- removed copper zone on layer 1, net SW_5V
- removed copper zone on layer 16, net SW_5V
- removed copper zone on layer 1, net SW_5V1
- removed copper zone on layer 16, net SW_5V1
- removed copper zone on layer 1, net VIN
Other:
- board size 160 x 100 mm -> 88.2 x 39 mm
- board text added: "+"
- board text added: "-"
