File: Tractive System Light Control Board.brd (EAGLE design)
At the start: 88.2 x 39 mm, 57 parts, among them J1 WM9811CT-ND, J2 WM9811CT-ND, T1 750313734, T2 LMC555, U1 ISO7221, U12 SN6501DBVR, U2 TPS562219, U21 LM1085IS, U3 LM139, U36 LTC1155, U37 CSD17506Q5A, U4 SN74LVC1G00DRL

Commit message: Made changes, about to start finishing layout
Parts:
- removed C10, C72, C73: 10uF, adafruit:C0805
- removed LED2: GREEN, FormE:CHIPLED_0805
- removed LED3: RED, FormE:CHIP-LED0805
- removed R13: 20k, adafruit:R0805
- removed R14: 10.5k, adafruit:R0805
- removed R17: 1K, adafruit:R0805
- removed T2: LMC555, FormE:LMC555
- removed U21: LM1085IS, FormE:TO-263
- removed U4: SN74LVC1G00DRL, FormE:LITTLE_LOGIC_BASIC_DRL
- added C11, C14, C15, C46: 0.1uF, rcl:C0805
- added C16: 0.1uF, adafruit:C0805
- added C17: 10uF, adafruit:C0805
- added J3, J4: MOLEX_CLICKMATE-2-VERTICAL, FormE:MOLEX-CLIKMATE-2-VERTICAL-HEADER
- added R6: (no value), FormE:TO-220-2
- added R8: 20k, adafruit:R0805
- added R9: 1K, adafruit:R0805
- added T3: LMC555, FormE:LMC555
- added U$1, U$2: 581002B02500G, FormE:AAVID-581X
- added U38: LM124, FormE:D14
- C1: device adafruit:C0805 -> rcl:C0805
- J1, J2: value WM9811CT-ND -> MOLEX_CLICKMATE-2-VERTICAL
- LED1: value (none) -> GREEN; device FormE:SMARTLED-TTW -> FormE:CHIPLED_0805
- R1: value 1K -> (none); device adafruit:R0805 -> FormE:TO-220-2
- R10: value 10k -> 1.2k
- R11: value 47k -> 10k
- R18: value 140k -> 271k
- R19, R21, R22: value 120k -> 271k
- R20: value 10k -> 10.5k
- R23: value 10k -> 100k
- R7: value 1k -> 10k
- U3: value LM139 -> SN74LVC1G00DRL; device FormE:D14 -> FormE:LITTLE_LOGIC_BASIC_DRL
- moved R1 165.8 mm to (-60.3, -105.4), turned to 0 degrees
- moved U3 155.9 mm to (-62.9, -141.6)
- moved R20 152.7 mm to (-62.9, -125.1), turned to 0 degrees
- moved C1 84.9 mm to (69.2, 8.89)
- moved LED1 63.4 mm to (-10.8, -14.6), turned to 0 degrees
- moved R7 14.6 mm to (1.27, -5.08)
- moved R50 6.63 mm to (57.8, 15.2), turned to 270 degrees
- moved TP21 6.38 mm to (64.1, 17.1)
- moved U36 6.38 mm to (63.5, 12.7)
- moved U37 6.38 mm to (69.2, 14.0)
- moved TP22 6.25 mm to (60.3, 17.1)
- moved U12 2.54 mm to (48.3, 36.2)
Connections:
- net TSAL_SUPPLY renamed TSAL_CONTROL
- removed net +12V: C73.1, LED2.A, U21.2, U21.GND, U21.GND1, U36.1, U36.6, U37.5, U37.6, U37.7, U37.8, U37.PAD, U37.PAD1, U37.VIA1, U37.VIA2, U37.VIA3, U37.VIA4, U37.VIA5, U37.VIA6, U37.VIA7, U37.VIA8, U37.VIA9
- removed net N$15: C10.1, R13.1, T2.2, T2.6
- removed net N$16: LED1.C@1, R17.2
- removed net N$5: R13.2, R14.1, T2.7
- removed net N$9: T2.4, U4.4
- new net 555_TIMER_CONTROL: T3.4, U3.4
- new net HV_INDICATOR_SIGNAL_LV: U1.P$6, U3.1
- new net N$10: J3.2, R6.P$2
- new net N$12: R20.1, R8.2, T3.7
- net +5V: now also C11.1, C14.1, C16.1, R20.2, T3.8, U3.5; no longer C1.1, R14.2, T2.8, U4.5
- net +5V/1: now also C15.1, C46.1, R9.2, U38.4; no longer R20.1, U3.3
- net 555_TIMER_OUTPUT: now also T3.3; no longer LED1.A@1, T2.3
- net AIR_CLOSED: now also U3.2; no longer U4.2
- net BATT_V_REFERENCE: now also U38.9; no longer U3.7
- net GND: now also C11.2, C14.2, C15.2, C16.2, C17.2, T3.1, U3.3; no longer C10.2, C72.2, C73.2, R1.1, R17.1, T2.1, U21.1, U4.3
- net GND1: now also C46.2, R6.P$1, U38.11; no longer U3.12
- net HV_INDICATOR_SIGNAL_HV: now also LED1.C, R7.2, U38.8; no longer LED3.C, R20.2, U3.1
- net N$13: now also C17.1, R8.1, T3.2, T3.6; no longer LED2.C, R1.2
- net N$4: now also LED1.A, R9.1; no longer U1.P$6, U4.1
- net N$48: now also U38.10; no longer U3.6
- net N$7: now also J4.1, R1.P$2; no longer LED3.A, R7.2
- net V+: now also R1.P$1
- net VCC: now also C1.1, U36.1, U36.6, U37.5, U37.6, U37.7, U37.8, U37.PAD, U37.PAD1, U37.VIA1, U37.VIA2, U37.VIA3, U37.VIA4, U37.VIA5, U37.VIA6, U37.VIA7, U37.VIA8, U37.VIA9; no longer C72.1, U21.3
Routing:
- net AIR_CLOSED: track 46.0 -> 0.00 mm, vias 2 -> 0
- net HV_INDICATOR_SIGNAL_HV: track 26.2 -> 7.59 mm
- net N$5: track 11.5 -> 0.00 mm
- net 555_TIMER_OUTPUT: track 37.9 -> 30.1 mm, vias 3 -> 2
- net HV_INDICATOR_SIGNAL_LV: track 0.00 -> 5.82 mm
- net +5V: track 5.05 -> 9.07 mm, vias 22 -> 15
- net N$16: track 3.13 -> 0.00 mm
- net N$13: track 2.56 -> 0.00 mm
- net N$31: track 4.93 -> 7.47 mm
- net TSAL_CONTROL: track 2.17 -> 4.60 mm
- net VCC: track 3.02 -> 5.45 mm
- net GND: track 16.5 -> 15.2 mm, vias 37 -> 29
- net N$40: track 4.93 -> 3.86 mm
- net GND1: track 35.8 -> 36.8 mm
- net +12V: track 0.93 -> 0.00 mm, vias 12 -> 0
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- removed copper zone on layer 1, net +12V
- removed copper zone on layer 15, net +12V
- removed copper zone on layer 1, net 12V_CURRENT_SENSE+
- removed copper zone on layer 1, net 555_TIMER_SUPPLY
Other:
- board size 88.2 x 39 mm -> 101.6 x 39 mm
