File: Tractive System Light Control Board.sch (EAGLE design)
At the start: 70 parts, among them J1 MOLEX_CLICKMATE-2-VERTICAL, J2 MOLEX_CLICKMATE-2-VERTICAL, Q1 BSS138, T1 750313734, U1 ISO7221, U12 SN6501DBVR, U2 TPS562219, U21 LM1085IS, U3 SN74LVC1G04DRL, U36 LTC1155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

Commit message: Reconfigured the schematic to improve functionality and readability
Parts:
- removed C18: 100uF, rcl:C-USC0805
- removed LED4, LED6, LED7, LED8: (no value), FormE:LED
- removed Q1: BSS138, FormE:BSS138
- removed R12: 10k, rcl:R-US_R0805
- removed R15: 0.33k, adafruit:R-US_R0805
- removed R16, R9: 1K, adafruit:R-US_R0805
- removed R24: 10, adafruit:R-US_R0805
- removed R6: 0.007, adafruit:R-US_R0805
- removed TP1: PTR1B1,27, testpad:PTR1B1,27
- removed U38: LM124, FormE:LM124
- removed U6: LTC1155, FormE:LTC1155
- removed U8: CSD17506Q5A, FormE:CSD17506Q5A
- removed U9: SN74LVC1G86DRL, FormE:LL_X-OR:SN74LVC1G86DRL
- added C1: 0.1uF, adafruit:C-USC0805
- added LED3: (no value), FormE:LEDCHIP-LED0805
- added R7: 10k, adafruit:R-US_R0805
- added U4: SN74LVC1G00DRL, FormE:LL_NAND:SN74LVC1G00DRL
- J1, J2: value MOLEX_CLICKMATE-2-VERTICAL -> WM9811CT-ND
- R10: value 1.2k -> 10k
- R11: value 10k -> 47k
- R18: value 10k -> 140k
- R19, R21, R22: value 10k -> 120k
- T2: value (none) -> LMC555
- U3: value SN74LVC1G04DRL -> LM139; device FormE:LL_INVERTER:SN74LVC1G04DRL -> FormE:LM139
Connections:
- net LED_CONTROL_12V renamed TSAL_SUPPLY
- removed net 12V_CURRENT_SENSE+: C73.1, R6.1, U21.OUT
- removed net 555_TIMER_SUPPLY: R14.1, R16.2, T2.+V, U8.S
- removed net AMS_CONTACTOR_INVERTED: H1.4, U9A.2
- removed net HV_INDICATOR_SIGNAL_LV: U1.INA, U9A.1
- removed net N$15 (its old number): C18.2, T2.CNT
- removed net N$19: R16.1, T2.RST
- removed net N$20: R15.1, T2.OUT
- removed net N$21: LED4.C, R9.2
- removed net N$22: LED4.A, LED6.C
- removed net N$24: LED6.A, LED7.C
- removed net N$25: LED7.A, LED8.C
- removed net N$35: U38C.OUT, U3A.IN
- removed net N$49: Q1.G, R24.1
- removed net N$60: Q1.D, R9.1
- removed net N$8: U6A.G, U8.G
- new net AIR_CLOSED: H1.4, U4A.IN2
- new net N$4: U1.OUTB, U4A.IN1
- new net N$7: LED3.A, R7.2
- net +12V: now also C73.1, U21.OUT; no longer R6.2
- net +5V: now also C1.1, R14.1, T2.+V, U4G$2.VCC; no longer U6A.D, U6P.VCC, U8.D, U9P.VCC
- net +5V/1: now also R7.1, U3P.VCC; no longer LED8.A, U38G$1.V+, U3G$2.VCC
- net 555_TIMER_OUTPUT: now also T2.OUT; no longer R15.2
- net BATT_V_REFERENCE: now also U3A.+; no longer U38C.+
- net GND: now also C1.2, U4G$2.GND; no longer C18.1, R12.1, U6P.GND, U9P.GND
- net GND1: now also U3P.GND; no longer Q1.S, U38G$1.V-, U3G$2.GND
- net HV_INDICATOR_SIGNAL_HV: now also LED3.C, U1.INB; no longer R24.2, U1.OUTA
- net N$48: now also U3A.-; no longer U38C.-
- net N$9: now also T2.RST, U4A.OUT; no longer R12.2, TP1.TP, U6A.IN, U9A.3
Other:
- note added: "0v when more than 52.5v is present 5v when less than 52.5v is present"
- note added: "Activates the TSAL timer if TS voltage is above 52.5v or either AIR is closed"
- note added: "Astable 555 Timer"
- note added: "Digital Isolator"
- note added: "ISOLATED TRACTIVE SYSTEM SECTION"
- note added: "Isolated DC to DC Converter"
- note added: "NEGATIVE TERMINAL"
- note added: "POSITIVE TERMINAL"
- note removed: "555 Timer Astable"
- note removed: "Batterie Voltage"
- note removed: "DC to DC Isolated Supply"
- note removed: "Divides battery voltage by 11.8"
- note removed: "HIgh Voltage"
- note removed: "HV MSIC."
- note removed: "HV indicator"
- note removed: "High Side FET-FET Driver"
- note removed: "ISOLATED POWER SUPPLY"
- note removed: "If signal from HV indicator or AMS, Then supply +5V to 555 Timer"
- note removed: "Isolator"
- note removed: "LV MSIC."
- note removed: "Pulls to ground when the main input is below ~54V"
- note removed: "TSAL Activation Logic"
- note removed: "TSAL Control Board"
- note removed: "Turns on an indicator when the voltage ouside the contactors is above ~60V"
- moved on the sheet: C11, C2, C3, C4, C5, C6, C7, C72, C73, C8, C9, H1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

Commit message: Changed RC values for 555 timer
Parts:
- removed C11: 100uF, adafruit:CPOL-USF
- added C10: 10uF, adafruit:C-USC0805
- LED3: value (none) -> RED
- R13: value 2k -> 20k
- R14: value 1.05k -> 10.5k
- R7: value 10k -> 1k
Connections:
- net +5V: now also R14.2; no longer R14.1
- net GND: now also C10.2; no longer C11.-
- net N$15: now also C10.1; no longer C11.+
- net N$5: now also R14.1; no longer R14.2
Other:
- moved on the sheet: C2, C3, C4, C5, C6, C7, C72, C73, C8, C9, L1, LED2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

Commit message: Made changes, about to start finishing layout
Parts:
- removed C10, C72, C73: 10uF, adafruit:C-USC0805
- removed LED2: GREEN, FormE:LEDCHIPLED_0805
- removed LED3: RED, FormE:LEDCHIP-LED0805
- removed R13: 20k, adafruit:R-US_R0805
- removed R14: 10.5k, adafruit:R-US_R0805
- removed R17: 1K, adafruit:R-US_R0805
- removed T2: LMC555, FormE:LMC555DGK
- removed U21: LM1085IS, FormE:LM1085
- removed U4: SN74LVC1G00DRL, FormE:LL_NAND:SN74LVC1G00DRL
- added C11, C14, C15, C46: 0.1uF, rcl:C-USC0805
- added C16: 0.1uF, adafruit:C-USC0805
- added C17: 10uF, adafruit:C-USC0805
- added J3, J4: MOLEX_CLICKMATE-2-VERTICAL, FormE:MOLEX_CLICKMATE-2-VERTICAL
- added R6: RTO020F10001JTE3, FormE:RTO020F10001JTE3
- added R8: 20k, adafruit:R-US_R0805
- added R9: 1K, adafruit:R-US_R0805
- added T3: LMC555, FormE:LMC555DGK
- added U$1, U$2: 581002B02500G, FormE:AAVID-581X
- added U38: LM124, FormE:LM124
- C1: device adafruit:C-USC0805 -> rcl:C-USC0805; MPN (none) -> C1005X7R1E104K050BB; OC_NEWARK (none) -> 04X3227; PARTNO GRM21BR61E106KA73L -> GRM21BR71E104KA01L
- J1, J2: value WM9811CT-ND -> MOLEX_CLICKMATE-2-VERTICAL
- LED1: value (none) -> GREEN; device FormE:LED -> FormE:LEDCHIPLED_0805; PARTNO (none) -> 598-8170-107F
- R1: value 1K -> RTO020F10001JTE3; device adafruit:R-US_R0805 -> FormE:RTO020F10001JTE3; PARTNO ERJ-6ENF1001V -> (none)
- R10: value 10k -> 1.2k
- R11: value 47k -> 10k
- R18: value 140k -> 271k
- R19, R21, R22: value 120k -> 271k
- R20: value 10k -> 10.5k; PARTNO ERJ-6ENF1002V -> ERJ-6ENF1051V
- R23: value 10k -> 100k
- R7: value 1k -> 10k
- U3: value LM139 -> SN74LVC1G00DRL; device FormE:LM139 -> FormE:LL_NAND:SN74LVC1G00DRL
Connections:
- net TSAL_SUPPLY renamed TSAL_CONTROL
- removed net +12V: C73.1, LED2.A, U21.OUT, U36A.D, U36P.VCC, U37.D
- removed net N$15: C10.1, R13.1, T2.THD, T2.TRG
- removed net N$16: LED1.C, R17.2
- removed net N$5: R13.2, R14.1, T2.DSC
- removed net N$9: T2.RST, U4A.OUT
- new net 555_TIMER_CONTROL: T3.RST, U3A.OUT
- new net HV_INDICATOR_SIGNAL_LV: U1.OUTB, U3A.IN1
- new net N$10: J3.2, R6.P$2
- new net N$12: R20.1, R8.2, T3.DSC
- net +5V: now also C11.1, C14.1, C16.1, R20.2, T3.+V, U3G$2.VCC; no longer C1.1, R14.2, T2.+V, U4G$2.VCC
- net +5V/1: now also C15.1, C46.1, R9.2, U38G$1.V+; no longer R20.1, U3P.VCC
- net 555_TIMER_OUTPUT: now also T3.OUT; no longer LED1.A, T2.OUT
- net AIR_CLOSED: now also U3A.IN2; no longer U4A.IN2
- net BATT_V_REFERENCE: now also U38C.-; no longer U3A.+
- net GND: now also C11.2, C14.2, C15.2, C16.2, C17.2, T3.GND, U3G$2.GND; no longer C10.2, C72.2, C73.2, R1.1, R17.1, T2.GND, U21.ADJ, U4G$2.GND
- net GND1: now also C46.2, R6.P$1, U38G$1.V-; no longer U3P.GND
- net HV_INDICATOR_SIGNAL_HV: now also LED1.C, R7.2, U38C.OUT; no longer LED3.C, R20.2, U3A.OUT
- net N$13: now also C17.1, R8.1, T3.THD, T3.TRG; no longer LED2.C, R1.2
- net N$4: now also LED1.A, R9.1; no longer U1.OUTB, U4A.IN1
- net N$48: now also U38C.+; no longer U3A.-
- net N$7: now also J4.1, R1.P$2; no longer LED3.A, R7.2
- net V+: now also R1.P$1
- net VCC: now also C1.1, U36A.D, U36P.VCC, U37.D; no longer C72.1, U21.IN
Other:
- note added: "555 Timer Astable"
- note added: "Ams Contactor Closed = 0 Open = 1"
- note added: "Divides battery voltage by 11.8"
- note added: "HV Battery Terminals"
- note added: "HV Measurment Point Connections"
- note added: "HV indicator"
- note added: "High Side FET-FET Driver"
- note added: "ISOLATED POWER SUPPLY"
- note added: "LV Connecter"
- note added: "Negative Terminal"
- note added: "TSAL Control Board"
- note added: "TSAL Powerstage"
- note added: "Turns on an indicator when the voltage ouside the contactors is above ~60V"
- note added: "Voltage Regulator"
- note removed: "Ams Contactor closed = 0 Open = 1"
- note removed: "Astable 555 Timer"
- note removed: "NEGATIVE TERMINAL"
- note removed: "Powerstage for TSAL"
- note removed: "REGULATED OUTPUT"
- note removed: "Voltage Regulators"
- moved on the sheet: C1, C2, C3, C4, C5, C6, C7, C8, C9, C90, C91, D33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
