File: Tractive System Light Control Board.sch (EAGLE design)
At the start: 131 parts, among them J2 MOLEX_CLICKMATE-2-VERTICAL, J3 MOLEX_CLICKMATE-2-VERTICAL, Q1 BSS138, Q100 FQD2N100, Q101 MMBT2222A, Q102 STP5N60M2, Q12 FQD3P50, Q5 BSS138, T1 WURTH-7491181112, U1 ISO7221, U10 TPS562219, U100 LM5022, U14 LM139, U2 TPS562219, U3 CD4069UB-SOIC, U36 LTC1155, U37 CSD17506Q5A, U4 CD4071B, U44 TL7712A-SOIC, U6 LTC1155, U8 CSD17506Q5A

Commit message: Added 55 Timer schematics and DC DC Converter
Parts:
- removed C33, C34: 0.1uF, adafruit:C-USC0805
- removed C35, C36: 1uF, rcl:C-USC0805
- removed Q5: BSS138, FormE:BSS138
- removed R53, R54: 10k, rcl:R-US_R0805
- removed R55: 100, rcl:R-US_R0805
- removed R56: 2.2K, rcl:R-US_R0805
- removed S2: TE-FSM4JSMATR, FormE:TE-FSM4JSMATR
- removed TP38, TP39, TP40: PTR1TP20R, testpad:PTR1TP20R
- removed U3: CD4069UB-SOIC, FormE:CD4069UB-SOIC
- removed U4: CD4071B, FormE:CD4071B
- removed U44: TL7712A-SOIC, FormE:TL7709A-SOIC
- added H3: (no value), FormE:MOLEX_MX120G
- added J4: MOLEX_CLICKMATE-2-VERTICAL, FormE:MOLEX_CLICKMATE-2-VERTICAL
- added U9: SN74LVC1G86, FormE:LL_X-OR:SN74LVC1G86
- J1: value (none) -> MOLEX_CLICKMATE-2-VERTICAL; device FormE:MOLEX-PICOLOCK-4PIN-504050-0491 -> FormE:MOLEX_CLICKMATE-2-VERTICAL
- T2: device FormE:ICM7555,56 -> FormE:LMC555DGK
Connections:
- net N$80 renamed 60V_CHECK
- removed net +3V3: Q5.G, R54.2, R56.1
- removed net AMS_DIGITAL_OV-12V: J1.1, U3A.IN
- removed net LED_CONTROL: TP20.TP, U37.S
- removed net MCU_RESET: C36.1, R55.1, R56.2, TP39.TP, U44.*RESIN
- removed net N$26: C33.2, U44.CT
- removed net N$27: C34.2, U44.REF
- removed net N$63: Q5.S, R54.1, U35C.IN
- removed net N$65: Q5.D, R53.1, TP38.TP, U44.*RESET
- removed net N$66: R55.2, S2.1, S2.2
- removed net POR: TP40.TP, U35C.OUT
- removed net VDD: C35.1, R53.2, U44.SENSE, U44.VCC
- new net AMS_CONTACTOR: J4.2
- new net LED_CONTROL_12V: H3.P10, H3.P11, H3.P12, H3.P7, H3.P8, H3.P9, TP20.TP, U37.S
- net +5V: no longer U3P.VCC
- net +5V/1: now also U9P.VCC; no longer U4P.VCC
- net AMS_DIGITAL_+12V_INVERTED_HV: now also U9A.2; no longer U4A.IN2
- net AMS_DIGITAL_+12V_INVERTED_LV: no longer U3A.OUT
- net GND: now also J3.2; no longer J1.3, U3P.GND
- net GND1: now also H3.P1, H3.P2, H3.P3, H3.P4, H3.P5, H3.P6, J2.1, U9P.GND; no longer C33.1, C34.1, C35.2, C36.2, S2.3, S2.4, U44.GND, U4P.GND
- net HV_INDICATOR_OUTPUT_+12V: now also U9A.1; no longer U4A.IN1
- net N$9: now also U9A.3; no longer U4A.OUT
- net V+: now also J1.1, J1.2; no longer J2.1
- net VCC: now also J3.1; no longer J1.2
Other:
- note added: "Ams Contactor closed = 0 Open = 1"
- note added: "From AMS"
- note added: "Use this connector??? Goes to TSAL, how sealed comming out of high junction Voltage box?"
- note added: "WH_supply"
- note removed: "LED_CONTROL"
- note removed: "N$80"
- note removed: "NEED????????"
- note removed: "Need special connector for high voltage?"
- moved on the sheet: J3

Commit message: Mid-design change, about to start deleting things
Parts:
- removed LED10, LED11, LED3, LED9: (no value), FormE:LED
- added LED4, LED6, LED7: (no value), FormE:LED
- added LED5: GREEN, FormE:LEDCHIPLED_0805
- added R18, R19, R21, R22, R23: 10k, adafruit:R-US_R0805
- added U3: SN74LVC1G04DRL, FormE:LL_INVERTER:SN74LVC1G04DRL
- added U38: LM124, FormE:LM124
- R2: value 54.9k -> 33.2K
- R9: value 100 -> 1K; PARTNO ERJ-6ENF1002V -> ERJ-6ENF1001V
- U9: value SN74LVC1G86 -> SN74LVC1G86DRL; device FormE:LL_X-OR:SN74LVC1G86 -> FormE:LL_X-OR:SN74LVC1G86DRL
Connections:
- net SW_5V1 renamed SW_5V2
- removed net N$46: LED8.A, LED9.C
- removed net N$47: R20.2, R24.2, U14C.OUT
- removed net N$50: LED10.A, LED11.C
- removed net N$51: LED10.C, LED9.A
- removed net N$52: LED11.A, R9.2
- new net +3V3: C7.1, C8.1, C9.1, L1.P$2, LED5.A, R2.2
- new net HV_INDICATOR_SIGNAL: R20.2, R24.2, U3A.OUT
- new net N$18: R18.2, R19.1
- new net N$21: LED4.C, R9.2
- new net N$22: LED4.A, LED6.C
- new net N$24: LED6.A, LED7.C
- new net N$25: LED7.A, LED8.C
- new net N$26: R19.2, R21.1
- new net N$27: R21.2, R22.1
- new net N$30: R22.2, R23.1
- new net N$35: U38C.OUT, U3A.IN
- net +5V: no longer C7.1, C8.1, C9.1, L1.P$2, LED3.A, R2.2
- net +5V/1: now also LED8.A, U3G$2.VCC
- net FILTERED_BATT_VOLTAGE_FB: now also U38C.+; no longer U14C.-
- net GND1: now also R23.2, U3G$2.GND
- net HV_INDICATOR_OUTPUT_+12V: no longer R9.1
- net N$2: now also LED5.C; no longer LED3.C
- net N$48: now also U38C.-; no longer U14C.+
- net N$60: now also R9.1; no longer LED8.C
- net V+: now also R18.1
Other:
- note added: "Voltage Filter"
- moved on the sheet: C2, C3, C4, C5, C6, C7, C8, C9, J3, J4, L1, LED8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

Commit message: Schematic Done
Parts:
- removed C1, C19, C20: 22uF, adafruit:C-USC0805
- removed C10: DNP, adafruit:C-USC0805K
- removed C100, C101: 0.047uF, adafruit:C-USC1812K
- removed C102: 0.022uF, adafruit:C-USC0805K
- removed C103: 4.7uF, adafruit:C-USC1210K
- removed C104: 1uF, adafruit:C-USC0805K
- removed C105: 680pF, adafruit:C-USC0805K
- removed C106: 330pF, adafruit:C-USC0805K
- removed C107: 6800pF, adafruit:C-USC0805K
- removed C111: 100uF, adafruit:CPOL-USF
- removed C12, C16: 0.1uF, adafruit:C-USC0805
- removed C121: 0.33uF, adafruit:C-USC0805K
- removed C13, C14: 10uF, adafruit:C-USC0805
- removed C15: 8200pF, adafruit:C-USC0805
- removed C17: 3.3uF, adafruit:C-USC1210K
- removed D100, D5: CMZ5931B, FormE:CMZ5931B
- removed D101: ES1D, FormE:ES1D
- removed D105, D3: BAV21W, FormE:BAV21W
- removed D110: CMZ5918B, FormE:CMZ5918B
- removed F1: 0805L020, FormE:0805L020
- removed F2: 0485.500DR, FormE:LITTELFUSE_485
- removed H3: (no value), FormE:MOLEX_MX120G
- removed J3, J4: MOLEX_CLICKMATE-2-VERTICAL, FormE:MOLEX_CLICKMATE-2-VERTICAL
- removed L2: 4.7uH, FormE:SRP6540
- removed Q100: FQD2N100, FormE:FQD2N100
- removed Q101: MMBT2222A, FormE:MMBT2222A
- removed Q102: STP5N60M2, FormE:STP3N150
- removed Q12: FQD3P50, FormE:FQD3P50
- removed R100, R101, R102, R103, R104, R105, R47: 1M, adafruit:R-US_R0805
- removed R106, R113: 20.5k, adafruit:R-US_R0805
- removed R107: 8.25k, adafruit:R-US_R0805
- removed R108: 499, adafruit:R-US_R0805
- removed R109: 1.05k, adafruit:R-US_R0805
- removed R110: 17.4k, adafruit:R-US_R0805
- removed R111: 2k, adafruit:R-US_R0805
- removed R112: 24.9, adafruit:R-US_R0805
- removed R114: 243k, adafruit:R-US_R0805
- removed R115: 0.82, adafruit:R-US_R1210
- removed R116: 2M, adafruit:R-US_R0805
- removed R117: 10k, adafruit:R-US_R1210
- removed R121: 205k, adafruit:R-US_R0805
- removed R25, R26: 10K, adafruit:R-US_R0805
- removed R27: 1K, adafruit:R-US_R0805
- removed R7: 4.7k, adafruit:R-US_R0805
- removed R8: 0, adafruit:R-US_R0805
- removed TP20: PTR1TP20R, testpad:PTR1TP20R
- removed U$1: AAVID-579302B00000G, FormE:AAVID-579302B00000G
- removed U10: TPS562219, FormE:TPS562219
- removed U100: LM5022, FormE:LM5022
- added C72, C73: 10uF, adafruit:C-USC0805
- added C90, C91: 10uF, rcl:C-USC1206
- added D33, D34: MBR0520LT3G, FormE:MBR0520LT3G
- added D35: MM3Z5V1B, FormE:MM3Z5V1B
- added H1: MOLEX_CLIKMATE-8-VERTICAL-5025841170, FormE:MOLEX_CLIKMATE-8-VERTICAL-5025841170
- added R72: 47R, rcl:R-US_R0805
- added TP2: PTR1TP20R, testpad:PTR1TP20R
- added U12: SN6501DBVR, FormE:SN6501
- added U21: LM1085IS, FormE:LM1085
- LED2: value (none) -> GREEN; device FormE:LED -> FormE:LEDCHIPLED_0805; PARTNO (none) -> 598-8170-107F
- R1: value 54.9k -> 1K; PARTNO ERA-6AEB5492V -> ERJ-6ENF1001V
- R2: value 33.2K -> 54.9K
- R6: value 470k -> 0.007; PARTNO RC0805FR-07470KL -> PMR10EZPFU7L00
- T1: value WURTH-7491181112 -> 750313734; device FormE:WURTH-7491181112 -> FormE:WURTH-750313734
Connections:
- removed net +3V3: C7.1, C8.1, C9.1, L1.P$2, LED5.A, R2.2
- removed net 60V_CHECK: C100.1, C101.1, D5.CATHODE, Q12.S, R100.2, R103.2, R106.2, R6.2, T1.1
- removed net AMS_CONTACTOR: J4.2
- removed net AMS_DIGITAL_+12V_INVERTED_HV: U9A.2
- removed net AMS_DIGITAL_+12V_INVERTED_LV: U1.INB
- removed net BATT_VOLTAGE_FB: R6.1, R7.2, R8.1
- removed net COMP: C106.1, R107.1, U100.COMP
- removed net CS: R109.1, R116.2, U100.CS
- removed net FB: C106.2, C107.2, R110.1, R111.2, U100.FB
- removed net FILTERED_BATT_VOLTAGE_FB: C10.1, R8.2, U38C.+
- removed net HV_INDICATOR_OUTPUT_+12V: U9A.1
- removed net HV_INDICATOR_SIGNAL: R20.2, R24.2, U3A.OUT
- removed net N$10: R103.1, R104.2, R116.1
- removed net N$11: R104.1, R105.2
- removed net N$12: R101.1, R102.2
- removed net N$14: C121.1, D110.CATHODE, Q101.B, R102.1, R121.2
- removed net N$23: R26.2, U10.EN
- removed net N$28: LED2.C, R27.2
- removed net N$29: D105.ANODE, R112.1
- removed net N$30: R22.2, R23.1
- removed net N$32: Q102.S, R108.2, R115.2
- removed net N$33: Q102.D, T1.5
- removed net N$34: C105.1, R108.1, R109.2
- removed net N$37: Q100.D, R106.1
- removed net N$38: D101.ANODE, T1.6
- removed net N$4: D105.CATHODE, D3.ANODE, R110.2
- removed net N$7: R100.1, R101.2
- removed net N$81: D5.ANODE, Q12.G, R47.2
- removed net N$82: D101.CATHODE, F1.P$1
- removed net N$83: F2.P$2, Q12.D
- removed net OUT: Q102.G, U100.OUT
- removed net RT: R114.2, U100.RT
- removed net SS: C102.1, U100.SS
- removed net SS_5V: C15.1, U10.SS
- removed net SW_5V: C16.2, L2.P$1, U10.SW
- removed net UVLO: Q101.E, R113.2, U100.UVLO
- removed net VBST_5V: C16.1, U10.VBST
- removed net VFB_5V: R1.1, R25.2, U10.VFB
- removed net VIN: C103.1, D3.CATHODE, Q100.S, Q101.C, U100.VIN
- new net 12V_CURRENT_SENSE+: C73.1, R6.1, U21.OUT
- new net AMS_CONTACTOR_INVERTED: H1.8, U9A.2
- new net BATT_V_REFERENCE: R22.2, R23.1, U38C.+
- new net HV_INDICATOR_SIGNAL_HV: R20.2, R24.2, U1.OUTA, U3A.OUT
- new net HV_INDICATOR_SIGNAL_LV: U1.INA, U9A.1
- new net N$40: T1.3, U12.D1
- new net N$41: D33.A, T1.6
- new net N$43: C90.1, D33.K, D34.K, R72.1
- new net N$45: D34.A, T1.4
- net +12V: now also LED2.A, R6.2; no longer C111.+, C17.1, F1.P$2, R112.2, R117.2
- net +5V: now also C7.1, C8.1, C9.1, L1.P$2, LED5.A, R2.2, T1.2, U1.VCC2, U12.VCC; no longer U1.VCC1
- net +5V/1: now also C91.1, D35.CATHODE, R72.2, U1.VCC1; no longer C1.1, C19.1, C20.1, L2.P$2, LED2.A, R1.2, U1.VCC2
- net GND: now also C72.2, C73.2, H1.2, H1.5, H1.6, R1.1, U1.GND2, U12.GND, U21.ADJ; no longer C1.2, C12.2, C13.2, C14.2, C19.2, C20.2, J3.2, R27.1, U1.GND1
- net GND1: now also C90.2, C91.2, D35.ANODE, T1.5, U1.GND1; no longer C10.2, C100.2, C101.2, C102.2, C103.2, C104.2, C105.2, C111.-, C121.2, C15.2, C17.2, D100.ANODE, D110.ANODE, H3.P1, H3.P2, H3.P3, H3.P4, H3.P5, H3.P6, R111.1, R113.1, R114.1, R115.1, R117.1, R121.1, R25.1, R47.1, R7.1, T1.9, U1.GND2, U10.GND, U100.GND
- net LED_CONTROL_12V: now also H1.3, H1.4, TP2.TP; no longer H3.P10, H3.P11, H3.P12, H3.P7, H3.P8, H3.P9, TP20.TP
- net N$13: now also LED2.C, R1.2; no longer D100.CATHODE, Q100.G, R105.1
- net N$31: now also T1.1, U12.D2; no longer C107.1, R107.2
- net V+: no longer F2.P$1
- net VCC: now also C72.1, H1.7, U21.IN; no longer C104.1, C12.1, C13.1, C14.1, J3.1, R26.1, U10.VIN, U100.VCC
Other:
- note added: "DC to DC Isolated Supply"
- note added: "Divides battery voltage by 11.8"
- note added: "HIgh Voltage"
- note added: "HV MSIC."
- note added: "ISOLATED POWER SUPPLY"
- note added: "Isolator"
- note added: "LV MSIC."
- note added: "Powerstage for TSAL"
- note added: "REGULATED OUTPUT"
- note added: "TSAL Activation Logic"
- note added: "TSAL Control Board"
- note added: "Voltage Regulators"
- note removed: "555_TIMER_OUTPUT"
- note removed: "555_TIMER_SUPPLY"
- note removed: "AMS_DIGITAL_+12V_INVERTED_HV"
- note removed: "AMS_DIGITAL_+12V_INVERTED_LV"
- note removed: "Feedback"
- note removed: "From AMS"
- note removed: "Fuse (500mA)"
- note removed: "HV_INDICATOR_OUTPUT_+12V"
- note removed: "High Volt Flyback Converter"
- note removed: "Powerstage for light"
- note removed: "Reverse voltage protection"
- note removed: "Startup Circuit"
- note removed: "Steps down batterie voltage to filtered batterie voltage"
- note removed: "Supplies 12V to the tractive system side of the board, power comes from the TS battery"
- note removed: "Use this connector??? Goes to TSAL, how sealed comming out of high junction Voltage box?"
- note removed: "Voltage Filter"
- note removed: "WH_supply"
- moved on the sheet: C11, C18, C2, C3, C4, C5, C6, C7, C8, C9, J1, J2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

Commit message: Layout Done: Need graphic for HV, maybe logo in bottom right corner?
Parts:
- removed U14: LM139, FormE:LM139
- removed U35: (no value), FormE:SN74LVC04ASOIC
Connections:
- net +12V: no longer U35POWER.VCC
- net +5V: now also R50.2, U6A.D, U6P.VCC, U8.D, U9P.VCC
- net +5V/1: now also U38G$1.V+; no longer R50.2, U14P.VCC, U6A.D, U6P.VCC, U8.D, U9P.VCC
- net AMS_CONTACTOR_INVERTED: now also H1.4; no longer H1.8
- net GND: now also C11.-, C18.1, H1.8, R12.1, R17.1, T2.GND, U36P.GND, U6P.GND, U9P.GND; no longer H1.6
- net GND1: now also U38G$1.V-; no longer C11.-, C18.1, R12.1, R17.1, T2.GND, U14P.GND, U35POWER.GND, U36P.GND, U6P.GND, U9P.GND
- net LED_CONTROL_12V: now also H1.6, H1.7; no longer H1.3, H1.4
- net VCC: now also H1.1; no longer H1.7
Other:
- moved on the sheet: C11, C18, C2, C3, C4, C5, C6, C7, C72, C73, C8, C9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

Commit message: Added resistors and heat sink to schematic, about to make changes
Parts:
- removed C72, C73: 10uF, adafruit:C-USC0805
- removed LED2: GREEN, FormE:LEDCHIPLED_0805
- removed LED4, LED6, LED7, LED8: (no value), FormE:LED
- removed R20: 10k, adafruit:R-US_R0805
- removed U21: LM1085IS, FormE:LM1085
- removed U3: SN74LVC1G04DRL, FormE:LL_INVERTER:SN74LVC1G04DRL
- removed U8: CSD17506Q5A, FormE:CSD17506Q5A
- added C1, C10, C12, C13, C14, C15, C46: 0.1uF, rcl:C-USC0805
- added J3, J4: MOLEX_CLICKMATE-2-VERTICAL, FormE:MOLEX_CLICKMATE-2-VERTICAL
- added L3: GREEN, FormE:LEDCHIPLED_0805
- added Q2: BSS138, FormE:BSS138
- added R7: 10k, adafruit:R-US_R0805
- added U$1, U$2: 581002B02500G, FormE:AAVID-581X
- added U4: (no value), FormE:SN74LVC04ASOIC
- LED1: value (none) -> GREEN; device FormE:LED -> FormE:LEDCHIPLED_0805; PARTNO (none) -> 598-8170-107F
- R1: value 1K -> RTO020F10001JTE3; device adafruit:R-US_R0805 -> FormE:RTO020F10001JTE3; PARTNO ERJ-6ENF1001V -> (none)
- R18, R19, R21, R22: value 10k -> 271k
- R23: value 10k -> 100k
- R6: value 0.007 -> RTO020F10001JTE3; device adafruit:R-US_R0805 -> FormE:RTO020F10001JTE3; PARTNO PMR10EZPFU7L00 -> (none)
Connections:
- removed net +12V: LED2.A, R6.2, U36A.D, U36P.VCC, U37.D
- removed net 12V_CURRENT_SENSE+: C73.1, R6.1, U21.OUT
- removed net N$13: LED2.C, R1.2
- removed net N$21: LED4.C, R9.2
- removed net N$22: LED4.A, LED6.C
- removed net N$24: LED6.A, LED7.C
- removed net N$25: LED7.A, LED8.C
- removed net N$35: U38C.OUT, U3A.IN
- new net AMS_CONTACTOR: H1.4, U4D.IN
- new net N$10: J3.2, R6.P$2
- new net N$4: LED1.C, R9.2
- new net N$7: J4.1, R1.P$2
- net +5V: now also C10.1, C12.1, C13.1, C14.1, Q2.D, U4POWER.VCC; no longer U8.D
- net +5V/1: now also C15.1, C46.1, LED1.A, R7.1; no longer LED8.A, R20.1, U3G$2.VCC
- net 555_TIMER_OUTPUT: now also L3.A; no longer LED1.A
- net 555_TIMER_SUPPLY: now also Q2.S; no longer U8.S
- net AMS_CONTACTOR_INVERTED: now also U4D.OUT, U9A.1; no longer H1.4, U9A.2
- net BATT_V_REFERENCE: now also U38C.-; no longer U38C.+
- net GND: now also C1.2, C10.2, C12.2, C13.2, C14.2, C15.2, U4POWER.GND; no longer C72.2, C73.2, R1.1, U21.ADJ
- net GND1: now also C46.2, R6.P$1; no longer U3G$2.GND
- net HV_INDICATOR_SIGNAL_HV: now also R7.2, U1.INB, U38C.OUT; no longer R20.2, U1.OUTA, U3A.OUT
- net HV_INDICATOR_SIGNAL_LV: now also U1.OUTB, U9A.2; no longer U1.INA, U9A.1
- net N$16: now also L3.C; no longer LED1.C
- net N$48: now also U38C.+; no longer U38C.-
- net N$8: now also Q2.G; no longer U8.G
- net V+: now also R1.P$1
- net VCC: now also C1.1, U36A.D, U36P.VCC, U37.D; no longer C72.1, U21.IN
Other:
- note removed: "REGULATED OUTPUT"
- moved on the sheet: C11, C18, C2, C3, C4, C5, C6, C7, C8, C9, C90, C91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

Commit message: Fixed small schematic errors, about to start layout
Parts:
- removed C10, C12, C13: 0.1uF, rcl:C-USC0805
- removed C18: 100uF, rcl:C-USC0805
- removed L3: GREEN, FormE:LEDCHIPLED_0805
- removed Q1, Q2: BSS138, FormE:BSS138
- removed R12: 10k, rcl:R-US_R0805
- removed R13: 2k, adafruit:R-US_R0805
- removed R14: 1.05k, adafruit:R-US_R0805
- removed R15: 0.33k, adafruit:R-US_R0805
- removed R16, R17: 1K, adafruit:R-US_R0805
- removed R24: 10, adafruit:R-US_R0805
- removed T2: (no value), FormE:LMC555DGK
- removed TP1: PTR1B1,27, testpad:PTR1B1,27
- removed U4: (no value), FormE:SN74LVC04ASOIC
- removed U6: LTC1155, FormE:LTC1155
- removed U9: SN74LVC1G86DRL, FormE:LL_X-OR:SN74LVC1G86DRL
- added C16: 0.1uF, adafruit:C-USC0805
- added C17: 10uF, adafruit:C-USC0805
- added R20: 10.5k, adafruit:R-US_R0805
- added R8: 20k, adafruit:R-US_R0805
- added T3: LMC555, FormE:LMC555DGK
- added U3: SN74LVC1G00DRL, FormE:LL_NAND:SN74LVC1G00DRL
- C11: value 100uF -> 0.1uF; device adafruit:CPOL-USF -> rcl:C-USC0805; MPN (none) -> C1005X7R1E104K050BB; OC_NEWARK (none) -> 04X3227; PARTNO EEE-1EA101XP -> GRM21BR71E104KA01L
Connections:
- net LED_CONTROL_12V renamed TSAL_CONTROL
- removed net 555_TIMER_SUPPLY: Q2.S, R14.1, R16.2, T2.+V
- removed net AMS_CONTACTOR: H1.4, U4D.IN
- removed net AMS_CONTACTOR_INVERTED: U4D.OUT, U9A.1
- removed net N$15: C18.2, T2.CNT
- removed net N$16: L3.C, R17.2
- removed net N$19: R16.1, T2.RST
- removed net N$20: R15.1, T2.OUT
- removed net N$49: Q1.G, R24.1
- removed net N$5: R13.2, R14.2, T2.DSC
- removed net N$6: C11.+, R13.1, T2.THD, T2.TRG
- removed net N$60: Q1.D, R9.1
- removed net N$8: Q2.G, U6A.G
- removed net N$9: R12.2, TP1.TP, U6A.IN, U9A.3
- new net 555_TIMER_CONTROL: T3.RST, U3A.OUT
- new net AIR_CLOSED: H1.4, U3A.IN2
- new net N$12: R20.1, R8.2, T3.DSC
- new net N$13: C17.1, R8.1, T3.THD, T3.TRG
- net +5V: now also C11.1, C16.1, R20.2, T3.+V, U3G$2.VCC; no longer C10.1, C12.1, C13.1, Q2.D, U4POWER.VCC, U6A.D, U6P.VCC, U9P.VCC
- net +5V/1: now also R9.2; no longer LED1.A
- net 555_TIMER_OUTPUT: now also T3.OUT; no longer L3.A, R15.2
- net GND: now also C11.2, C16.2, C17.2, T3.GND, U3G$2.GND; no longer C10.2, C11.-, C12.2, C13.2, C18.1, R12.1, R17.1, T2.GND, U4POWER.GND, U6P.GND, U9P.GND
- net GND1: no longer Q1.S
- net HV_INDICATOR_SIGNAL_HV: now also LED1.C; no longer R24.2
- net HV_INDICATOR_SIGNAL_LV: now also U3A.IN1; no longer U9A.2
- net N$4: now also LED1.A, R9.1; no longer LED1.C, R9.2
Other:
- note added: "0v when more than 52.5v is present 5v when less than 52.5v is present"
- note added: "Activates the TSAL timer if TS voltage is above 52.5v or either AIR is closed"
- note added: "Ams Contactor Closed = 0 Open = 1"
- note added: "Digital Isolator"
- note added: "HV Battery Terminals"
- note added: "HV Measurment Point Connections"
- note added: "ISOLATED TRACTIVE SYSTEM SECTION"
- note added: "Isolated DC to DC Converter"
- note added: "LV Connector"
- note added: "Negative Terminal"
- note added: "POSITIVE TERMINAL"
- note added: "TSAL Powerstage"
- note added: "Voltage Regulator"
- note removed: "Ams Contactor closed = 0 Open = 1"
- note removed: "Batterie Voltage"
- note removed: "DC to DC Isolated Supply"
- note removed: "HIgh Voltage"
- note removed: "HV MSIC."
- note removed: "If signal from HV indicator or AMS, Then supply +5V to 555 Timer"
- note removed: "Isolator"
- note removed: "LV MSIC."
- note removed: "Powerstage for TSAL"
- note removed: "Pulls to ground when the main input is below ~54V"
- note removed: "TSAL Activation Logic"
- note removed: "Voltage Regulators"
- moved on the sheet: C1, C14, C15, C2, C3, C4, C46, C5, C6, C7, C8, C9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

Commit message: Done with layout, about to start BOM
Parts:
- removed LED1: GREEN, FormE:LEDCHIPLED_0805
- removed R10: 1.2k, adafruit:R-US_R0805
- removed R11: 10k, adafruit:R-US_R0805
- removed U38: LM124, FormE:LM124
- added C10: 0.1uF, rcl:C-USC0805
- added L2: GREEN, FormE:LEDCHIPLED_0805
- added R12, R13: 10k, adafruit:R-US_R0805
- added U4: LM139, FormE:LM139
- added U5: MAX6168AESA+, FormE:MAX616X
- R18, R19, R21, R22: value 271k -> 150K
- R23: value 100k -> 10K
Connections:
- removed net N$10: J3.2, R6.P$2
- removed net N$48: R10.1, R11.2, U38C.+
- removed net V+: J1.1, J1.2, R1.P$1, R18.1
- new net 0.9V_REF: R12.2, R13.1, U4A.-
- new net 1.8V_REF: C10.1, R12.1, U5.OUT
- new net B+: J1.2, R1.P$1, R18.1
- new net B-: J2.1, R23.2, R6.P$2
- new net N$6: J3.2, R6.P$1
- net +5V/1: now also U4P.VCC, U5.IN; no longer R11.1, U38G$1.V+
- net AIR_CLOSED: now also H1.7; no longer H1.4
- net BATT_V_REFERENCE: now also U4A.+; no longer U38C.-
- net GND: no longer C15.2
- net GND1: now also C10.2, C15.2, R13.2, U4P.GND, U5.GND; no longer J2.1, J2.2, R10.2, R23.2, R6.P$1, U38G$1.V-
- net HV_INDICATOR_SIGNAL_HV: now also L2.C, U4A.OUT; no longer LED1.C, U38C.OUT
- net N$4: now also L2.A; no longer LED1.A
- net TSAL_CONTROL: now also H1.3, H1.4; no longer H1.6, H1.7
Other:
- note added: "0.9V Voltage Reference"
- moved on the sheet: C1, C11, C14, C15, C16, C17, C2, C3, C4, C46, C5, C6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

Commit message: BOM Done, files next
Parts:
- removed C90, C91: 10uF, rcl:C-USC1206
- added C12, C13: 10uF, rcl:C-USC0805
- D33, D34: PARTNO (none) -> MBR0520LT3G
- D35: PARTNO (none) -> MM3Z3V3T1G
- H1: PARTNO (none) -> 5025841170
- R1, R6: PARTNO (none) -> RTO020F10001JTE3
- R32: value 47R -> 47; PARTNO (none) -> ERJ-6ENF1000V
- T1: PARTNO (none) -> 750313734
- T3: PARTNO (none) -> LMC555CM/NOPB
- U1: PARTNO (none) -> ISO7221CDR
- U12: PARTNO (none) -> SN6501DBVR
- U3: PARTNO (none) -> SN74LVC1G00DRLR
- U4: PARTNO (none) -> LM139DR
- U5: PARTNO (none) -> MAX6168AESA+
- renumbered R72 to R32, TP2 to TP1
Connections:
- net +5V/1: now also C13.1; no longer C91.1
- net GND1: now also C12.2, C13.2; no longer C90.2, C91.2
- net N$43: now also C12.1; no longer C90.1
