File: Tractive System Light Control Board.sch (EAGLE design)
At the start: 63 parts, among them J1 MOLEX_CLICKMATE-2-VERTICAL, J2 MOLEX_CLICKMATE-2-VERTICAL, J3 MOLEX_CLICKMATE-2-VERTICAL, J4 MOLEX_CLICKMATE-2-VERTICAL, T1 750313734, T3 LMC555, U1 ISO7221, U12 SN6501DBVR, U2 TPS562219, U3 SN74LVC1G00DRL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

Commit message: BOM Done, about to generate files
Parts:
- C12, C13: PARTNO GRM21BR71E104KA01L -> GRM21BR61E106KA73L
- C16: PARTNO GRM21BR61E106KA73L -> 08053C104KAT2A
- R8: PARTNO ERJ-6ENF2001V -> ERJ-3EKF2002V
Connections:
- removed net B-: J2.1, R23.2, R6.P$2
- net GND1: now also J2.1, R23.2, R6.P$2
Changed lines of the file:
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@@
 </part>
 <part name="R8" library="adafruit" deviceset="R-US_" device="R0805" value="20k">
-<attribute name="PARTNO" value="ERJ-6ENF2001V"/>
+<attribute name="PARTNO" value="ERJ-3EKF2002V"/>
 </part>
 <part name="R20" library="adafruit" deviceset="R-US_" device="R0805" value="10.5k">
@@
 <part name="GND21" library="supply1" deviceset="GND" device=""/>
 <part name="C16" library="adafruit" deviceset="C-US" device="C0805" value="0.1uF">
-<attribute name="PARTNO" value="GRM21BR61E106KA73L"/>
+<attribute name="PARTNO" value="08053C104KAT2A"/>
 </part>
 <part name="GND22" library="supply1" deviceset="GND" device=""/>
@@
 <attribute name="MPN" value="C1005X7R1E104K050BB"/>
 <attribute name="OC_NEWARK" value="04X3227"/>
-<attribute name="PARTNO" value="GRM21BR71E104KA01L"/>
+<attribute name="PARTNO" value="GRM21BR61E106KA73L"/>
 </part>
 <part name="C13" library="rcl" deviceset="C-US" device="C0805" value="10uF">
@@
 <attribute name="MPN" value="C1005X7R1E104K050BB"/>
 <attribute name="OC_NEWARK" value="04X3227"/>
-<attribute name="PARTNO" value="GRM21BR71E104KA01L"/>
+<attribute name="PARTNO" value="GRM21BR61E106KA73L"/>
 </part>
 <part name="TP1" library="testpad" deviceset="PTR1" device="TP20R"/>
@@
 <attribute name="PARTNO" value="ERJ-6ENF1000V"/>
 </part>
+<part name="SUPPLY13" library="supply2" deviceset="GND1" device=""/>
 </parts>
 <sheets>
@@
 <attribute name="PARTNO" x="281.94" y="38.1" size="1.778" layer="96" display="off"/>
 </instance>
+<instance part="SUPPLY13" gate="G$1" x="109.22" y="93.98"/>
 </instances>
 <busses>
@@
 <pinref part="SUPPLY12" gate="G$1" pin="GND1"/>
 <wire x1="182.88" y1="30.48" x2="182.88" y2="33.02" width="0.1524" layer="91"/>
+</segment>
+<segment>
+<pinref part="R23" gate="G$1" pin="2"/>
+<wire x1="109.22" y1="99.06" x2="109.22" y2="101.6" width="0.1524" layer="91"/>
+<wire x1="109.22" y1="99.06" x2="101.6" y2="99.06" width="0.1524" layer="91"/>
+<wire x1="101.6" y1="99.06" x2="99.06" y2="99.06" width="0.1524" layer="91"/>
+<wire x1="22.86" y1="124.46" x2="99.06" y2="124.46" width="0.1524" layer="91"/>
+<wire x1="99.06" y1="124.46" x2="99.06" y2="99.06" width="0.1524" layer="91"/>
+<label x="73.66" y="127" size="1.778" layer="95"/>
+<pinref part="J2" gate="G$1" pin="1"/>
+<wire x1="101.6" y1="93.98" x2="101.6" y2="99.06" width="0.1524" layer="91"/>
+<junction x="101.6" y="99.06"/>
+<pinref part="R6" gate="G$1" pin="P$2"/>
+<wire x1="22.86" y1="121.92" x2="22.86" y2="124.46" width="0.1524" layer="91"/>
+<pinref part="SUPPLY13" gate="G$1" pin="GND1"/>
+<wire x1="109.22" y1="96.52" x2="109.22" y2="99.06" width="0.1524" layer="91"/>
+<junction x="109.22" y="99.06"/>
 </segment>
 </net>
@@
 </segment>
 </net>
-<net name="B-" class="0">
-<segment>
-<pinref part="R23" gate="G$1" pin="2"/>
-<wire x1="109.22" y1="99.06" x2="109.22" y2="101.6" width="0.1524" layer="91"/>
-<wire x1="109.22" y1="99.06" x2="101.6" y2="99.06" width="0.1524" layer="91"/>
-<wire x1="101.6" y1="99.06" x2="99.06" y2="99.06" width="0.1524" layer="91"/>
-<wire x1="22.86" y1="124.46" x2="99.06" y2="124.46" width="0.1524" layer="91"/>
-<wire x1="99.06" y1="124.46" x2="99.06" y2="99.06" width="0.1524" layer="91"/>
-<label x="73.66" y="127" size="1.778" layer="95"/>
-<pinref part="J2" gate="G$1" pin="1"/>
-<wire x1="101.6" y1="93.98" x2="101.6" y2="99.06" width="0.1524" layer="91"/>
-<junction x="101.6" y="99.06"/>
-<pinref part="R6" gate="G$1" pin="P$2"/>
-<wire x1="22.86" y1="121.92" x2="22.86" y2="124.46" width="0.1524" layer="91"/>
-</segment>
-</net>

Commit message: Fixed BOM, added MM3Z5V1B
Parts:
- D35: PARTNO MM3Z3V3T1G -> MM3Z5V1B
- R18, R19, R21, R22: PARTNO ERJ-6ENF1002V -> ERJ-6ENF1503V
- R20: PARTNO ERJ-6ENF1051V -> ERA-8ARW1052V
- R32: PARTNO ERJ-6ENF1000V -> ERJ-6ENF4702V
Changed lines of the file:
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@@
 </part>
 <part name="R18" library="adafruit" deviceset="R-US_" device="R0805" value="150K">
-<attribute name="PARTNO" value="ERJ-6ENF1002V"/>
+<attribute name="PARTNO" value="ERJ-6ENF1503V"/>
 </part>
 <part name="R19" library="adafruit" deviceset="R-US_" device="R0805" value="150K">
-<attribute name="PARTNO" value="ERJ-6ENF1002V"/>
+<attribute name="PARTNO" value="ERJ-6ENF1503V"/>
 </part>
 <part name="R21" library="adafruit" deviceset="R-US_" device="R0805" value="150K">
-<attribute name="PARTNO" value="ERJ-6ENF1002V"/>
+<attribute name="PARTNO" value="ERJ-6ENF1503V"/>
 </part>
 <part name="R22" library="adafruit" deviceset="R-US_" device="R0805" value="150K">
-<attribute name="PARTNO" value="ERJ-6ENF1002V"/>
+<attribute name="PARTNO" value="ERJ-6ENF1503V"/>
 </part>
 <part name="R23" library="adafruit" deviceset="R-US_" device="R0805" value="10K">
@@
 </part>
 <part name="D35" library="FormE" deviceset="MM3Z5V1B" device="" value="MM3Z5V1B">
-<attribute name="PARTNO" value="MM3Z3V3T1G"/>
+<attribute name="PARTNO" value="MM3Z5V1B"/>
 </part>
 <part name="GND40" library="supply1" deviceset="GND" device=""/>
@@
 </part>
 <part name="R20" library="adafruit" deviceset="R-US_" device="R0805" value="10.5k">
-<attribute name="PARTNO" value="ERJ-6ENF1051V"/>
+<attribute name="PARTNO" value="ERA-8ARW1052V"/>
 </part>
 <part name="P+16" library="supply1" deviceset="+5V" device=""/>
@@
 <part name="TP1" library="testpad" deviceset="PTR1" device="TP20R"/>
 <part name="R32" library="rcl" deviceset="R-US_" device="R0805" value="47">
-<attribute name="PARTNO" value="ERJ-6ENF1000V"/>
+<attribute name="PARTNO" value="ERJ-6ENF4702V"/>
 </part>
 <part name="SUPPLY13" library="supply2" deviceset="GND1" device=""/>

Commit message: Fixed comparator and BOM, about to generate files
Parts:
- R20: PARTNO ERA-8ARW1052V -> ERA-6AEB1052V
- R8: PARTNO ERJ-3EKF2002V -> ERA-6AEB204V
Connections:
- net 0.9V_REF: now also U4A.+; no longer U4A.-
- net BATT_V_REFERENCE: now also U4A.-; no longer U4A.+
Other:
- moved on the sheet: C1, C10, C11, C12, C13, C14, C15, C16, C17, C2, C3, C4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

Commit message: A few minor layout tweaks. Regenerated gerbers and BOM
Parts:
- H1: PARTNO 5025841170 -> 5025840870
- J1, J2, J3, J4: PARTNO (none) -> 5025840270
- R1, R6: value RTO020F10001JTE3 -> 10k
- R20: PARTNO ERA-6AEB1052V -> ERJ-6ENF1052V
- R32: PARTNO ERJ-6ENF4702V -> ERA-6AEB470V
- R8: PARTNO ERA-6AEB204V -> ERJ-6ENF2002V
Changed lines of the file:
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@@
 <?xml version="1.0" encoding="utf-8"?>
 <!DOCTYPE eagle SYSTEM "eagle.dtd">
-<eagle version="7.5.0">
+<eagle version="7.3.0">
 <drawing>
 <settings>
@@
 <attribute name="PARTNO" value="ISO7221CDR"/>
 </part>
-<part name="J2" library="FormE" deviceset="MOLEX_CLICKMATE-2-VERTICAL" device=""/>
+<part name="J2" library="FormE" deviceset="MOLEX_CLICKMATE-2-VERTICAL" device="">
+<attribute name="PARTNO" value="5025840270"/>
+</part>
 <part name="R50" library="rcl" deviceset="R-US_" device="R0805" value="DNP"/>
 <part name="U36" library="FormE" deviceset="LTC1155" device="">
@@
 <part name="TP21" library="testpad" deviceset="PTR1" device="TP20R"/>
 <part name="TP22" library="testpad" deviceset="PTR1" device="TP20R"/>
-<part name="J1" library="FormE" deviceset="MOLEX_CLICKMATE-2-VERTICAL" device=""/>
+<part name="J1" library="FormE" deviceset="MOLEX_CLICKMATE-2-VERTICAL" device="">
+<attribute name="PARTNO" value="5025840270"/>
+</part>
 <part name="C2" library="adafruit" deviceset="C-US" device="C0805" value="0.1uF">
 <attribute name="PARTNO" value="GRM21BR71E104KA01L"/>
@@
 <part name="SUPPLY2" library="supply2" deviceset="GND1" device=""/>
 <part name="H1" library="FormE" deviceset="MOLEX_CLIKMATE-8-VERTICAL-5025841170" device="" value="">
-<attribute name="PARTNO" value="5025841170"/>
+<attribute name="PARTNO" value="5025840870"/>
 </part>
 <part name="GND8" library="supply1" deviceset="GND" device=""/>
@@
 <attribute name="PARTNO" value="GRM21BR71E104KA01L"/>
 </part>
-<part name="J3" library="FormE" deviceset="MOLEX_CLICKMATE-2-VERTICAL" device=""/>
-<part name="J4" library="FormE" deviceset="MOLEX_CLICKMATE-2-VERTICAL" device=""/>
+<part name="J3" library="FormE" deviceset="MOLEX_CLICKMATE-2-VERTICAL" device="">
+<attribute name="PARTNO" value="5025840270"/>
+</part>
+<part name="J4" library="FormE" deviceset="MOLEX_CLICKMATE-2-VERTICAL" device="">
+<attribute name="PARTNO" value="5025840270"/>
+</part>
 <part name="U$1" library="FormE" deviceset="AAVID-581X" device="" value="581002B02500G">
 <attribute name="PARTNO" value="581002B02500G"/>
@@
 <attribute name="PARTNO" value="581002B02500G"/>
 </part>
-<part name="R1" library="FormE" deviceset="RTO020F10001JTE3" device="" value="">
+<part name="R1" library="FormE" deviceset="RTO020F10001JTE3" device="" value="10k">
 <attribute name="PARTNO" value="RTO020F10001JTE3"/>
 </part>
-<part name="R6" library="FormE" deviceset="RTO020F10001JTE3" device="" value="">
+<part name="R6" library="FormE" deviceset="RTO020F10001JTE3" device="" value="10k">
 <attribute name="PARTNO" value="RTO020F10001JTE3"/>
 </part>
@@
 </part>
 <part name="R8" library="adafruit" deviceset="R-US_" device="R0805" value="20k">
-<attribute name="PARTNO" value="ERA-6AEB204V"/>
+<attribute name="PARTNO" value="ERJ-6ENF2002V"/>
 </part>
 <part name="R20" library="adafruit" deviceset="R-US_" device="R0805" value="10.5k">
-<attribute name="PARTNO" value="ERA-6AEB1052V"/>
+<attribute name="PARTNO" value="ERJ-6ENF1052V"/>
 </part>
 <part name="P+16" library="supply1" deviceset="+5V" device=""/>
@@
 <part name="TP1" library="testpad" deviceset="PTR1" device="TP20R"/>
 <part name="R32" library="rcl" deviceset="R-US_" device="R0805" value="47">
-<attribute name="PARTNO" value="ERJ-6ENF4702V"/>
+<attribute name="PARTNO" value="ERA-6AEB470V"/>
 </part>
 <part name="SUPPLY13" library="supply2" deviceset="GND1" device=""/>
@@
 <attribute name="PARTNO" x="340.36" y="116.84" size="1.778" layer="96" display="off"/>
 </instance>
-<instance part="J2" gate="G$1" x="101.6" y="81.28" rot="R270"/>
+<instance part="J2" gate="G$1" x="101.6" y="81.28" rot="R270">
+<attribute name="PARTNO" x="101.6" y="81.28" size="1.778" layer="96" display="off"/>
+</instance>
 <instance part="R50" gate="G$1" x="467.36" y="38.1" rot="R90"/>
 <instance part="U36" gate="A" x="492.76" y="27.94"/>
@@
 <instance part="TP22" gate="G$1" x="474.98" y="25.4"/>
 <instance part="U36" gate="P" x="495.3" y="27.94"/>
-<instance part="J1" gate="G$1" x="101.6" y="177.8" rot="R90"/>
+<instance part="J1" gate="G$1" x="101.6" y="177.8" rot="R90">
+<attribute name="PARTNO" x="101.6" y="177.8" size="1.778" layer="96" display="off"/>
+</instance>
 <instance part="C2" gate="G$1" x="378.46" y="231.14">
 <attribute name="PARTNO" x="378.46" y="231.14" size="1.778" layer="96" display="off"/>
@@
 <attribute name="MPN" x="317.5" y="134.62" size="1.778" layer="96" display="off"/>
 </instance>
-<instance part="J3" gate="G$1" x="22.86" y="91.44" rot="R270"/>
-<instance part="J4" gate="G$1" x="25.4" y="154.94" rot="R90"/>
+<instance part="J3" gate="G$1" x="22.86" y="91.44" rot="R270">
+<attribute name="PARTNO" x="22.86" y="91.44" size="1.778" layer="96" display="off"/>
+</instance>
+<instance part="J4" gate="G$1" x="25.4" y="154.94" rot="R90">
+<attribute name="PARTNO" x="25.4" y="154.94" size="1.778" layer="96" display="off"/>
+</instance>
 <instance part="U$1" gate="G$1" x="12.7" y="129.54">
 <attribute name="PARTNO" x="12.7" y="129.54" size="1.778" layer="96" display="off"/>
@@
 </instance>
 <instance part="SUPPLY12" gate="G$1" x="185.42" y="127"/>
-<instance part="C12" gate="G$1" x="297.18" y="33.02" smashed="yes">
-<attribute name="NAME" x="298.196" y="33.655" size="1.778" layer="95"/>
+<instance part="C12" gate="G$1" x="297.18" y="33.02">
 <attribute name="PARTNO" x="297.18" y="33.02" size="1.778" layer="96" rot="R180" display="off"/>
 <attribute name="OC_NEWARK" x="297.18" y="33.02" size="1.778" layer="96" display="off"/>
@@
 <attribute name="MPN" x="297.18" y="33.02" size="1.778" layer="96" display="off"/>
 </instance>
-<instance part="C13" gate="G$1" x="274.32" y="33.02" smashed="yes">
-<attribute name="NAME" x="275.336" y="33.655" size="1.778" layer="95"/>
+<instance part="C13" gate="G$1" x="274.32" y="33.02">
 <attribute name="PARTNO" x="274.32" y="33.02" size="1.778" layer="96" rot="R180" display="off"/>
 <attribute name="OC_NEWARK" x="274.32" y="33.02" size="1.778" layer="96" display="off"/>

Commit message: Fixed 10k Resistors- TSAL Control Board V2.0- Ready To Order
Parts:
- R1, R6: value 10k -> RTO020F10001JTE3
Changed lines of the file:
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@@
 <?xml version="1.0" encoding="utf-8"?>
 <!DOCTYPE eagle SYSTEM "eagle.dtd">
-<eagle version="7.3.0">
+<eagle version="7.5.0">
 <drawing>
 <settings>
@@
 <attribute name="PARTNO" value="581002B02500G"/>
 </part>
-<part name="R1" library="FormE" deviceset="RTO020F10001JTE3" device="" value="10k">
+<part name="R1" library="FormE" deviceset="RTO020F10001JTE3" device="" value="">
 <attribute name="PARTNO" value="RTO020F10001JTE3"/>
 </part>
-<part name="R6" library="FormE" deviceset="RTO020F10001JTE3" device="" value="10k">
+<part name="R6" library="FormE" deviceset="RTO020F10001JTE3" device="" value="">
 <attribute name="PARTNO" value="RTO020F10001JTE3"/>
 </part>

Commit message: Updated BOM, ready to order... again
Parts:
- T3: PARTNO LMC555CM/NOPB -> LMC555CMM/NOPB
Changed lines of the file:
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@@
 <part name="GND19" library="supply1" deviceset="GND" device=""/>
 <part name="T3" library="FormE" deviceset="LMC555" device="DGK" value="LMC555">
-<attribute name="PARTNO" value="LMC555CM/NOPB"/>
+<attribute name="PARTNO" value="LMC555CMM/NOPB"/>
 </part>
 <part name="R8" library="adafruit" deviceset="R-US_" device="R0805" value="20k">
